Commit message: fix gripper in sapien

File: ocrtoc_task/urdf/ur5e.urdf (robot description, URDF)
Before this commit: robot ur5e, 31 links, 30 joints
Links:
- link robotiq_2f_85_left_driver: geometry collision mesh filename=package://robotiq_2f_85_gripper_visualization/legacy/meshes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 scale=0.001 0.001 0.001; visual mesh filename=package://robotiq_2f_85_gripper_visualization/legacy/meshes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 scale=0.001 0.001 0.001
Joints:
- removed joint robotiq_2f_85_left_follower_joint
- removed joint robotiq_2f_85_right_follower_joint
- added joint robotiq_2f_85_left_driver_mimic_joint: type revolute, parent robotiq_arg2f_base_link, child robotiq_2f_85_left_driver, origin xyz=0 -0.0306011 0.054904 rpy=0 0 3.14159265359, axis 1 0 0, limit lower=0 upper=0.8 effort=1000 velocity=2.0
- added joint robotiq_2f_85_right_driver_mimic_joint: type revolute, parent robotiq_arg2f_base_link, child robotiq_2f_85_right_driver, origin xyz=0 0.0306011 0.054904 rpy=0 0 0, axis 1 0 0, limit lower=0 upper=0.8 effort=1000 velocity=2.0, mimic joint=robotiq_2f_85_left_driver_joint multiplier=1 offset=0
- joint robotiq_2f_85_left_driver_joint: axis 1 0 0 -> 8.31983143e-08 -9.52063817e-01 3.05899474e-01; child robotiq_2f_85_left_driver -> robotiq_2f_85_left_pad; limit lower=0 upper=0.8 effort=1000 velocity=2.0 -> lower=0 upper=0.0448 effort=1000 velocity=2.0; origin xyz=0 -0.0306011 0.054904 rpy=0 0 3.14159265359 -> xyz=3.35276e-08 -0.0461303 0.137834 rpy=0 0 3.14; parent robotiq_arg2f_base_link -> robotiq_2f_85_base; type revolute -> prismatic
- joint robotiq_2f_85_left_pad_joint: child robotiq_2f_85_left_pad -> robotiq_2f_85_left_follower; origin xyz=0 -0.0220203446692936 0.03242 rpy=0 0 0 -> xyz=0 0.0220203446692936 -0.03242 rpy=0 0 0; parent robotiq_2f_85_left_follower -> robotiq_2f_85_left_pad
- joint robotiq_2f_85_right_driver_joint: axis 1 0 0 -> 8.31388445e-08 -9.52019331e-01 3.06037896e-01; child robotiq_2f_85_right_driver -> robotiq_2f_85_right_pad; limit lower=0 upper=0.8 effort=1000 velocity=2.0 -> lower=0 upper=0.0448 effort=1000 velocity=2.0; mimic joint=robotiq_2f_85_left_driver_joint multiplier=1 offset=0 -> (none); origin xyz=0 0.0306011 0.054904 rpy=0 0 0 -> xyz=3.35276e-08 0.0461303 0.137834 rpy=0 0 0; parent robotiq_arg2f_base_link -> robotiq_2f_85_base; type revolute -> prismatic
- joint robotiq_2f_85_right_pad_joint: child robotiq_2f_85_right_pad -> robotiq_2f_85_right_follower; origin xyz=0 -0.0220203446692936 0.03242 rpy=0 0 0 -> xyz=0 0.0220203446692936 -0.03242 rpy=0 0 0; parent robotiq_2f_85_right_follower -> robotiq_2f_85_right_pad
