Commit message: fix issue-9

File: description/robotiq_2f_85_gripper_visualization/urdf/robotiq_2f_85.urdf.xacro (robot description, xacro)
@@ -542,11 +542,11 @@
 				</plugin>
 				<plugin name="${name}_right_pad_joint_plugin" filename="libroboticsgroup_gazebo_mimic_joint_plugin.so">
-					<joint>${name}_right_pad_joint</joint>
-					<mimicJoint>${name}_right_follower_joint</mimicJoint>
+					<joint>${name}_right_follower_joint</joint>
+					<mimicJoint>${name}_right_pad_joint</mimicJoint>
 					<multiplier>0</multiplier>
 				</plugin>
 				<plugin name="${name}_left_pad_joint_plugin" filename="libroboticsgroup_gazebo_mimic_joint_plugin.so">
-					<joint>${name}_left_pad_joint</joint>
-					<mimicJoint>${name}_right_follower_joint</mimicJoint>
+					<joint>${name}_right_follower_joint</joint>
+					<mimicJoint>${name}_left_pad_joint</mimicJoint>
 					<multiplier>0</multiplier>
 				</plugin>

Commit message: update description files

File: description/robotiq_2f_85_gripper_visualization/urdf/robotiq_2f_85.urdf.xacro (robot description, xacro)
@@ -1,556 +1,556 @@
 <?xml version="1.0"?>
 <!--
-	Coordinate system convention for grippers:
-	The pin of the gripper is along the y-axis, and z-axis points up.
-	The resulting x-axis is considered the palm face, so +y is right, and -y is left for
-	a right-hand gripper, whatever that means in this gripper.
-	Coarse and precise models:
-	Two granularities for collision are provided, a coarse (default) for quick motion
-	planning purposes, and a precise for grasp simulation. This is selected with the
-	boolean parameter precise_collision = true/false (default to false)
-	In the same line, there is the adaptive_transmission parameter that might use
-	pure mimic joints (default and motion does not consider adaptation) for visualization
-	and update of real hw, and an implementation of the 5-bar transmission with
-	spring transmission for grasp simulation.
-	For grasp simulation, the file 2f85.gazebo.xacro sets additional parameters such as
-	material properties, and simulation parameters.
+  Coordinate system convention for grippers:
+  The pin of the gripper is along the y-axis, and z-axis points up.
+  The resulting x-axis is considered the palm face, so +y is right, and -y is left for
+  a right-hand gripper, whatever that means in this gripper.
+  Coarse and precise models:
+  Two granularities for collision are provided, a coarse (default) for quick motion
+  planning purposes, and a precise for grasp simulation. This is selected with the
+  boolean parameter precise_collision = true/false (default to false)
+  In the same line, there is the adaptive_transmission parameter that might use
+  pure mimic joints (default and motion does not consider adaptation) for visualization
+  and update of real hw, and an implementation of the 5-bar transmission with
+  spring transmission for grasp simulation.
+  For grasp simulation, the file 2f85.gazebo.xacro sets additional parameters such as
+  material properties, and simulation parameters.
 -->
 <robot xmlns:xacro="http://ros.org/wiki/xacro">
-	<xacro:include filename="$(find robotiq_2f_85_gripper_visualization)/urdf/inertias.urdf.xacro" />
-	<xacro:macro name="robotiq_2f_85" params="parent name precise_collision:=false adaptive_transmission:=false with_pads:=true *origin sim">
-		<!-- the ee link of gripper -->
-		<joint name="${parent}_${name}_ee_joint" type="fixed">
-			<origin xyz="0 0 0.1493" rpy="0 0 0"/>
-			<parent link="${name}_base"/>
-			<child link="${name}_ee_link"/>
-		</joint>
-		<link name="${name}_ee_link"/>
-		<!-- base -->
-		<joint name="${parent}_${name}_base_joint" type="fixed">
-			<xacro:insert_block name="origin"/>
-			<parent link="${parent}"/>
-			<child link="${name}_base"/>
-		</joint>
-		<link name="${name}_base">
-			<inertial>
-				<mass value="0.5"/>
-				<origin xyz="0 0 ${0.015*0.5}"  />
-				<cylinder_inertia radius="0.04" length="0.045" mass="0.5"/>
-			</inertial>
-			<visual>
-				<origin xyz="0 0 0" rpy="0 -1.5708 0"/>
-				<geometry>
-					<mesh filename="package://robotiq_2f_85_gripper_visualization/meshes/visual/base.dae"/>
-				</geometry>
-			</visual>
-			<xacro:unless value="${precise_collision}">
-			<collision>
-				<origin xyz="0 0 0.015" rpy="0 0 0"/>
-				<geometry>
-					<cylinder radius="0.04" length="0.045"/>
-				</geometry>
-			</collision>
-			<collision>
-				<origin xyz="0 0 0.06" rpy="0 0 0"/>
-				<geometry>
-					<box size="0.03 0.03 0.06"/>
-				</geometry>
-			</collision>
-			</xacro:unless>
-			<xacro:if value="${precise_collision}">
-			<collision>
-				<geometry>
-					<mesh filename="package://robotiq_2f_85_gripper_visualization/meshes/collision/base.stl" scale="0.001 0.001 0.001"/>
-				</geometry>
-			</collision>
-			</xacro:if>
-		</link>
-		<!-- right finger -->
-		<joint name="${name}_right_driver_joint" type="revolute">
-			<origin xyz="0 0.0306011 0.054904" rpy="0 0 0"/>
-			<parent link="${name}_base"/>
-			<child link="${name}_right_driver"/>
-			<axis xyz="1 0 0"/>
-			<limit lower="${0 * 3.141592 / 180}" upper="${50 * 3.141592 / 180}" effort="60" velocity="${110 * 3.141592 / 180}" />
-		</joint>
-		<link name="${name}_right_driver">
-			<inertial>
-				<mass value="0.1"/>
-				<origin xyz="0 0.02 0" rpy="0 0 0" />
-				<box_inertia x_dim="0.02" y_dim="0.04" z_dim="0.02" mass="0.1"/>
-			</inertial>
-			<visual>
-				<geometry>
-					<mesh filename="package://robotiq_2f_85_gripper_visualization/meshes/visual/driver.dae" scale="0.001 0.001 0.001"/>
-				</geometry>
-			</visual>
-			<xacro:unless value="${precise_collision}">
-			<collision>
-				<origin xyz="0 0.01 0" rpy="-0.1 0 0"/>
-				<geometry>
-					<box size="0.002 0.004 0.002"/>
-				</geometry>
-			</collision>
-			</xacro:unless>
-			<xacro:if value="${precise_collision}">
-			<collision>
-				<geometry>
-					<mesh filename="package://robotiq_2f_85_gripper_visualization/meshes/collision/driver.stl" scale="0.001 0.001 0.001"/>
-				</geometry>
-			</collision>
-			</xacro:if>
-		</link>
-		<xacro:unless value="${adaptive_transmission}">
-		<joint name="${name}_right_coupler_joint" type="fixed">
-			<origin xyz="0 0.0315 -0.0041" rpy="0 0 0"/>
-			<parent link="${name}_right_driver"/>
-			<child link="${name}_right_coupler"/>
-		</joint>
-		</xacro:unless>
-		<xacro:if value="${adaptive_transmission}">
-			<joint name="${name}_right_coupler_joint" type="revolute">
-			<origin xyz="0 0.0315 -0.0041" rpy="0 0 0"/>
-			<parent link="${name}_right_driver"/>
-			<child link="${name}_right_coupler"/>
-			<axis xyz="1 0 0"/>
-			<limit lower="${-170 * 3.141592 / 180}" upper="${170 * 3.141592 / 180}" effort="176" velocity="${110 * 3.141592 / 180}" />
-		</joint>
-		</xacro:if>
-		<link name="${name}_right_coupler">
-			<inertial>
-				<mass value="0.1"/>
-				<origin xyz="0 0.0 0.025" rpy="-1.7 0 0"/>
-				<box_inertia x_dim="0.03" y_dim="0.065" z_dim="0.02" mass="0.1"/>
-			</inertial>
-			<visual>
-				<geometry>
-					<mesh filename="package://robotiq_2f_85_gripper_visualization/meshes/visual/coupler.dae" scale="0.001 0.001 0.001"/>
-				</geometry>
-			</visual>
-			<xacro:unless value="${precise_collision}">
-			<collision>
-				<origin xyz="0 0.0 0.025" rpy="-1.7 0 0"/>
-				<geometry>
-					<box size="0.03 0.065 0.02"/>
-				</geometry>
-			</collision>
-			</xacro:unless>
-			<xacro:if value="${precise_collision}">
-				<collision>
-					<geometry>
-						<mesh filename="package://robotiq_2f_85_gripper_visualization/meshes/collision/coupler.stl" scale="0.001 0.001 0.001"/>
-					</geometry>
-				</collision>
-			</xacro:if>
-		</link>
-		<joint name="${name}_right_follower_joint" type="revolute">
-			<origin xyz="0 0.0061 0.0471" rpy="0 0 0"/>
-			<parent link="${name}_right_coupler"/>
-			<child link="${name}_right_follower"/>
-			<axis xyz="1 0 0"/>
-			<limit lower="${-170 * 3.141592 / 180}" upper="${170 * 3.141592 / 180}" effort="176" velocity="${110 * 3.141592 / 180}" />
-			<xacro:unless value="${adaptive_transmission}">
-			<mimic joint="${name}_right_driver_joint" multiplier="-1"/>
-			</xacro:unless>
-		</joint>
-		<link name="${name}_right_follower">
-			<inertial>
-				<mass value="0.1"/>
-				<origin xyz="0 -0.018 0.022" />
-				<box_inertia x_dim="0.02" y_dim="0.015" z_dim="0.048" mass="0.1"/>
-			</inertial>
-			<visual>
-				<geometry>
-					<mesh filename="package://robotiq_2f_85_gripper_visualization/meshes/visual/follower.dae" scale="0.001 0.001 0.001"/>
-				</geometry>
-			</visual>
-			<xacro:unless value="${precise_collision}">
-			<collision>
-				<origin xyz="0 -0.01 0.022" rpy="0 0 0"/>
-				<geometry>
-					<box size="0.002 0.0015 0.0048"/>
-				</geometry>
-			</collision>
-			</xacro:unless>
-			<xacro:if value="${precise_collision}">
-			<collision>
-				<geometry>
-					<mesh filename="package://robotiq_2f_85_gripper_visualization/meshes/collision/follower.stl" scale="0.001 0.001 0.001"/>
-				</geometry>
-			</collision>
-			</xacro:if>
-		</link>
-		<xacro:if value="${with_pads}">
-			<joint name="${name}_right_pad_joint" type="revolute">
-				<parent link="${name}_right_follower"/>
-				<child link="${name}_right_pad"/>
-				<axis xyz="0 0 1"/>
-				<limit lower="0" upper="0" effort="200" velocity="0" />
-				<xacro:unless value="${adaptive_transmission}">
-				<mimic joint="${name}_right_driver_joint" multiplier="0"/>
-				</xacro:unless>
-			</joint>
-			<link name="${name}_right_pad">
-				<inertial>
-					<mass value="0.1"/>
-					<origin xyz="0 -0.022 0.031" />
-					<box_inertia x_dim="0.02" y_dim="0.008" z_dim="0.036" mass="0.1"/>
-				</inertial>
-				<visual>
-					<geometry>
-						<mesh filename="package://robotiq_2f_85_gripper_visualization/meshes/visual/pad.dae" scale="0.001 0.001 0.001"/>
-					</geometry>
-				</visual>
-				<xacro:unless value="${precise_collision}">
-				<collision>
-					<origin xyz="0 -0.022 0.031" rpy="0 0 0"/>
-					<geometry>
-						<box size="0.02 0.008 0.036"/>
-					</geometry>
-				</collision>
-				</xacro:unless>
-				<xacro:if value="${precise_collision}">
-				<collision>
-					<geometry>
-						<mesh filename="package://robotiq_2f_85_gripper_visualization/meshes/collision/pad.stl" scale="0.001 0.001 0.001"/>
-					</geometry>
-				</collision>
-				</xacro:if>
-			</link>
-		</xacro:if>
-		<joint name="${name}_right_spring_link_joint" type="revolute">
-			<origin xyz="0 0.012 0.0614" rpy="0 0 0"/>
-			<parent link="${name}_base"/>
-			<child link="${name}_right_spring_link"/>
-			<axis xyz="1 0 0"/>
-			<limit lower="${-170 * 3.141592 / 180}" upper="${170 * 3.141592 / 180}" effort="176" velocity="${110 * 3.141592 / 180}" />
-			<xacro:unless value="${adaptive_transmission}">
-			<mimic joint="${name}_right_driver_joint" multiplier="1"/>
-			</xacro:unless>
-		</joint>
-		<link name="${name}_right_spring_link">
-			<inertial>
-				<mass value="0.1"/>
-				<origin xyz="0 0.018 0.018" rpy="-0.7068 0 0"/>
-				<box_inertia x_dim="0.04" y_dim="0.02" z_dim="0.065" mass="0.1"/>
-			</inertial>
-			<visual>
-				<geometry>
-					<mesh filename="package://robotiq_2f_85_gripper_visualization/meshes/visual/spring_link.dae" scale="0.001 0.001 0.001"/>
-				</geometry>
-			</visual>
-			<xacro:unless value="${precise_collision}">
-			<collision>
-				<origin xyz="0 0.025 0.015" rpy="-0.7068 0 0"/>
-				<geometry>
-					<box size="0.004 0.002 0.0065"/>
-				</geometry>
-			</collision>
-			</xacro:unless>
-			<xacro:if value="${precise_collision}">
-			<collision>
-				<geometry>
-					<mesh filename="package://robotiq_2f_85_gripper_visualization/meshes/collision/spring_link.stl" scale="0.001 0.001 0.001"/>
-				</geometry>
-			</collision>
-			</xacro:if>
-		</link>
-		<!-- left finger -->
-		<joint name="${name}_left_driver_joint" type="revolute">
-			<origin xyz="0 -0.0306011 0.054904" rpy="0 0 3.141592653589793"/>
-			<parent link="${name}_base"/>
-			<child link="${name}_left_driver"/>
-			<axis xyz="1 0 0"/>
-			<limit lower="${0 * 3.141592 / 180}" upper="${50 * 3.141592 / 180}" effort="176" velocity="${110 * 3.141592 / 180}" />
-			<xacro:unless value="${adaptive_transmission}">
-			<mimic joint="${name}_right_driver_joint" multiplier="1"/>
-			</xacro:unless>
-		</joint>
-		<link name="${name}_left_driver">
-			<inertial>
-				<mass value="0.1"/>
-				<origin xyz="0 0.02 0" rpy="0 0 0" />
-				<box_inertia x_dim="0.02" y_dim="0.04" z_dim="0.02" mass="0.1"/>
-			</inertial>
-			<visual>
-				<geometry>
-					<mesh filename="package://robotiq_2f_85_gripper_visualization/meshes/visual/driver.dae" scale="0.001 0.001 0.001"/>
-				</geometry>
-			</visual>
-			<xacro:unless value="${precise_collision}">
-			<collision>
-				<origin xyz="0 0.01 0" rpy="-0.1 0 0"/>
-				<geometry>
-					<box size="0.002 0.004 0.002"/>
-				</geometry>
-			</collision>
-			</xacro:unless>
-			<xacro:if value="${precise_collision}">
-			<collision>
-				<geometry>
-					<mesh filename="package://robotiq_2f_85_gripper_visualization/meshes/collision/driver.stl" scale="0.001 0.001 0.001"/>
-				</geometry>
-			</collision>
-			</xacro:if>
-		</link>
-		<xacro:unless value="${adaptive_transmission}">
-		<joint name="${name}_left_coupler_joint" type="fixed">
-			<origin xyz="0 0.0315 -0.0041" rpy="0 0 0"/>
-			<parent link="${name}_left_driver"/>
-			<child link="${name}_left_coupler"/>
-		</joint>
-		</xacro:unless>
-		<xacro:if value="${adaptive_transmission}">
-			<joint name="${name}_left_coupler_joint" type="revolute">
-			<origin xyz="0 0.0315 -0.0041" rpy="0 0 0"/>
-			<parent link="${name}_left_driver"/>
-			<child link="${name}_left_coupler"/>
-			<axis xyz="1 0 0"/>
-			<limit lower="${-170 * 3.141592 / 180}" upper="${170 * 3.141592 / 180}" effort="176" velocity="${110 * 3.141592 / 180}" />
-		</joint>
-		</xacro:if>
-		<link name="${name}_left_coupler">
-			<inertial>
-				<mass value="0.1"/>
-				<origin xyz="0 0.0 0.025" rpy="-1.7 0 0"/>
-				<box_inertia x_dim="0.03" y_dim="0.065" z_dim="0.02" mass="0.1"/>
-			</inertial>
-			<visual>
-				<geometry>
-					<mesh filename="package://robotiq_2f_85_gripper_visualization/meshes/visual/coupler.dae" scale="0.001 0.001 0.001"/>
-				</geometry>
-			</visual>
-			<xacro:unless value="${precise_collision}">
-			<collision>
-				<origin xyz="0 0.0 0.025" rpy="-1.7 0 0"/>
-				<geometry>
-					<box size="0.03 0.065 0.02"/>
-				</geometry>
-			</collision>
-			</xacro:unless>
-			<xacro:if value="${precise_collision}">
-				<collision>
-					<geometry>
-						<mesh filename="package://robotiq_2f_85_gripper_visualization/meshes/collision/coupler.stl" scale="0.001 0.001 0.001"/>
-					</geometry>
-				</collision>
-			</xacro:if>
-		</link>
-		<joint name="${name}_left_follower_joint" type="revolute">
-			<origin xyz="0 0.0061 0.0471" rpy="0 0 0"/>
-			<parent link="${name}_left_coupler"/>
-			<child link="${name}_left_follower"/>
-			<axis xyz="1 0 0"/>
-			<limit lower="${-170 * 3.141592 / 180}" upper="${170 * 3.141592 / 180}" effort="176" velocity="${110 * 3.141592 / 180}" />
-			<xacro:unless value="${adaptive_transmission}">
-			<mimic joint="${name}_right_driver_joint" multiplier="-1"/>
-			</xacro:unless>
-		</joint>
-		<link name="${name}_left_follower">
-			<inertial>
-				<mass value="0.1"/>
-				<origin xyz="0 -0.018 0.022" />
-				<box_inertia x_dim="0.02" y_dim="0.015" z_dim="0.048" mass="0.1"/>
-			</inertial>
-			<visual>
-				<geometry>
-					<mesh filename="package://robotiq_2f_85_gripper_visualization/meshes/visual/follower.dae" scale="0.001 0.001 0.001"/>
-				</geometry>
-			</visual>
-			<xacro:unless value="${precise_collision}">
-			<collision>
-				<origin xyz="0 -0.01 0.022" rpy="0 0 0"/>
-				<geometry>
-					<box size="0.002 0.0015 0.0048"/>
-				</geometry>
-			</collision>
-			</xacro:unless>
-			<xacro:if value="${precise_collision}">
-			<collision>
-				<geometry>
-					<mesh filename="package://robotiq_2f_85_gripper_visualization/meshes/collision/follower.stl" scale="0.001 0.001 0.001"/>
-				</geometry>
-			</collision>
-			</xacro:if>
-		</link>
-		<xacro:if value="${with_pads}">
-			<joint name="${name}_left_pad_joint" type="revolute">
-				<parent link="${name}_left_follower"/>
-				<child link="${name}_left_pad"/>
-				<axis xyz="0 0 1"/>
-				<limit lower="0" upper="0" effort="200" velocity="0" />
-				<xacro:unless value="${adaptive_transmission}">
-				<mimic joint="${name}_right_driver_joint" multiplier="0"/>
-				</xacro:unless>
-			</joint>
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
File: description/robotiq_2f_85_gripper_visualization/urdf/robotiq_ur_coupler.urdf.xacro (robot description, xacro)
@@ -1,35 +1,35 @@
 <?xml version="1.0"?>
 <robot xmlns:xacro="http://ros.org/wiki/xacro">
-	<xacro:macro name="robotiq_ur_coupler" params="name parent">
-		<xacro:include filename="$(find robotiq_2f_85_gripper_visualization)/urdf/inertias.urdf.xacro" />
-		<joint name="${name}_coupler_joint" type="fixed">
-			<!-- total height of coupler, minus the depth of robot end-effector shape and the gripper small depth-->
-			<origin xyz="0 0 ${0.001*(13.5-3-3)}" rpy="0 0 0" />
-			<parent link="${parent}"/>
-			<child link="${name}"/>
-		</joint>
-		<link name="${name}">
-			<visual>
-				<origin xyz="0 0 ${-1*0.001*(13.93-3)*0.5}" rpy="0 0 0" />
-				<geometry>
-					<!-- only the visible part of the coupler -->
-					<cylinder length="${0.001*(13.9)}" radius="${0.5*0.075}" />
-				</geometry>
-				<material name="dark_grey">
-					<color rgba="0.05 0.05 0.05 1" />
-				</material>
-			</visual>
-			<collision>
-				<origin xyz="0 0 0" rpy="0 0 0" />
-				<geometry>
-					<cylinder length="${0.001*(13.5)}" radius="${0.5*0.075}" />
-				</geometry>
-			</collision>
-			<inertial>
-				<mass value="0.3"/>
-				<origin xyz="0 0 ${0.001*(13.9)*0.5}"  />
-				<cylinder_inertia radius="${0.5*0.075}" length="${0.001*(13.9)}" mass="0.3"/>
-			</inertial>
-		</link>
-	</xacro:macro>
+  <xacro:macro name="robotiq_ur_coupler" params="name parent">
+    <xacro:include filename="$(find robotiq_2f_85_gripper_visualization)/urdf/inertias.urdf.xacro" />
+    <joint name="${name}_coupler_joint" type="fixed">
+      <!-- total height of coupler, minus the depth of robot end-effector shape and the gripper small depth-->
+      <origin xyz="0 0 ${0.001*(13.5-3-3)}" rpy="0 0 0" />
+      <parent link="${parent}"/>
+      <child link="${name}"/>
+    </joint>
+    <link name="${name}">
+      <visual>
+        <origin xyz="0 0 ${-1*0.001*(13.93-3)*0.5}" rpy="0 0 0" />
+        <geometry>
+          <!-- only the visible part of the coupler -->
+          <cylinder length="${0.001*(13.9)}" radius="${0.5*0.075}" />
+        </geometry>
+        <material name="dark_grey">
+          <color rgba="0.05 0.05 0.05 1" />
+        </material>
+      </visual>
+      <collision>
+        <origin xyz="0 0 -0.008" rpy="0 0 0" />
+        <geometry>
+          <cylinder length="${0.001*(13.5)}" radius="${0.5*0.075}" />
+        </geometry>
+      </collision>
+      <inertial>
+        <mass value="0.3"/>
+        <origin xyz="0 0 ${0.001*(13.9)*0.5}"  />
+        <cylinder_inertia radius="${0.5*0.075}" length="${0.001*(13.9)}" mass="0.3"/>
+      </inertial>
+    </link>
+  </xacro:macro>
 </robot>

File: description/ur_e_description/urdf/ur5e.urdf.xacro (robot description, xacro)
@@ -2,5 +2,5 @@
 <robot xmlns:xacro="http://ros.org/wiki/xacro">
   <xacro:include filename="$(find ur_e_description)/urdf/ur.transmission.xacro" />
-  <xacro:include filename="$(find ur_e_description)/urdf/ur.gazebo.xacro" />
+  <!--xacro:include filename="$(find ur_e_description)/urdf/ur.gazebo.xacro" /-->
   <xacro:macro name="cylinder_inertial" params="radius length mass *origin">
     <inertial>
@@ -331,72 +331,6 @@
       </collision>
     </link>
-    <!-- Realsense Link -->
-  <xacro:include filename="$(find ur_e_description)/urdf/_d435.urdf.xacro" />
-  <sensor_d435 parent="${prefix}wrist_3_link">
-    <origin xyz="0.011013 0.094580 -0.10724" rpy="-3.1296068 0.028976 1.6645942"/>
-  </sensor_d435>
-    <!-- Kinect link -->
-    <material name="black">
-        <color rgba="0. 0. 0. 1" />
-    </material>
-    <material name="dark_grey">
-        <color rgba="0.1 0.1 0.1 1" />
-    </material>
-    <material name="grey">
-        <color rgba="0.6 0.6 0.6 1" />
-    </material>
-    <material name="white">
-        <color rgba="0.9 0.9 0.9 1" />
-    </material>
-    <joint name="kinect_camera_joint" type="fixed">
-      <origin rpy="0.1285134 0.8828308 -1.3433447" xyz="-0.13285 0.797229 0.58769"/>
-      <parent link="${prefix}base_link"/>
-      <child link="kinect_camera_visor" />
-    </joint>
-    <link name="kinect_camera_body">
-    <visual>
-      <origin xyz="0. 0. 0." />
-      <geometry>
-        <box size="0.0994 0.0996 0.023" />
-      </geometry>
-      <material name="white" />
-    </visual>
-  </link>
-    <link name="kinect_camera_base">
-    <visual>
-      <origin xyz="-0.013 0. 0." />
-      <geometry>
-        <box size="0.026 0.103 0.039" />
-      </geometry>
-      <material name="grey" />
-    </visual>
-    </link>
-    <link name="kinect_camera_visor">
-    <visual>
-      <origin xyz="-0.0128 0. 0." />
-      <geometry>
-        <box size="0.026 0.101 0.037" />
-      </geometry>
-      <material name="black" />
-    </visual>
-  </link>
-   <joint name="kinect_camera_base_to_body" type="fixed">
-    <parent link="kinect_camera_base" />
-    <child link="kinect_camera_body" />
-    <origin xyz="-0.0757 0. 0.008" rpy="0. 0. 0." />
-  </joint>
-  <joint name="kinect_camera_base_to_visor" type="fixed">
-    <parent link="kinect_camera_visor" />
-    <child link="kinect_camera_base" />
-    <origin xyz="0. 0. 0." rpy="0. 0. 0." />
-  </joint>
-  <joint name="kinect_optical_joint" type="fixed">
-      <origin xyz="0 0 0" rpy="${-M_PI/2} 0 ${-M_PI/2}" />
-      <parent link="kinect_camera_visor" />
-      <child link="kinect_optical_frame" />
-    </joint>
-  <link name="kinect_optical_frame"/>
     <xacro:ur_arm_transmission prefix="${prefix}" />
-    <xacro:ur_arm_gazebo prefix="${prefix}" />
+    <!--xacro:ur_arm_gazebo prefix="${prefix}" /-->
     <!-- ROS base_link to UR 'Base' Coordinates transform -->
     <link name="${prefix}base"/>
