Commit message: Update ur5e_joint_limited_robot.urdf.xacro

File: description/ur_e_description/urdf/ur5e_joint_limited_robot.urdf.xacro (robot description, xacro)
@@ -56,5 +56,5 @@
     <parent link="table" />
     <child link = "base_link" />
-    <origin xyz="0 -0.24 0.38" rpy="0.0 0.0 0" />
+    <origin xyz="0 -0.24 0.3875" rpy="0.0 0.0 0" />
   </joint>
   <!-- realsense tool -->
